File: Kicad/IDE.kicad_sch (KiCad schematic)
At the start: 14 parts, among them J2 LED, J3 IDE, U3 74HCT245, U4 74HCT245, U5 74HCT245

Commit message: PCB: Change IDE address line connections from A2-4 to A10-12 (Gayle vs AT-Apollo style IDE)
Connections:
- net A2 renamed A10
- net A3 renamed A11
- net A4 renamed A12
Changed lines of the file:
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@@
     (effects (font (size 1.27 1.27)) (justify right bottom))
   )
-  (label "A2" (at 80.01 151.765 180)
+  (label "A10" (at 80.01 151.765 180)
     (effects (font (size 1.27 1.27)) (justify right bottom))
   )
@@
     (effects (font (size 1.27 1.27)) (justify right bottom))
   )
-  (label "A4" (at 80.01 154.305 180)
+  (label "A12" (at 80.01 154.305 180)
     (effects (font (size 1.27 1.27)) (justify right bottom))
   )
@@
     (effects (font (size 1.27 1.27)) (justify right bottom))
   )
-  (label "A3" (at 80.01 156.845 180)
+  (label "A11" (at 80.01 156.845 180)
     (effects (font (size 1.27 1.27)) (justify right bottom))
   )

Commit message: PCB: Change IDE address line connections to A9-11 (AT-Bus style)
Parts:
- removed J3: IDE, Connector_IDC:IDC-Header_2x20_P2.54mm_Vertical, symbol Connector_Generic:Conn_02x20_Odd_Even
- added F1: Polyfuse 500mA Hold, Fuse:Fuse_1206_3216Metric, symbol Device:Polyfuse_Small
- added J3: Conn_02x22_Odd_Even, Connector_PinHeader_2.00mm:PinHeader_2x22_P2.00mm_Vertical, symbol Connector_Generic:Conn_02x22_Odd_Even
Connections:
- net A12 is gone; now on net A11: U5.15 (B3)
- net A10: now also U5.14 (B4); no longer U5.16 (B2)
- net A11: no longer U5.14 (B4)
- net B_D0: now also J3.4 (Pin_4)
- net B_D1: now also J3.6 (Pin_6)
- net B_D10: now also J3.13 (Pin_13)
- net B_D11: now also J3.11 (Pin_11)
- net B_D12: now also J3.9 (Pin_9)
- net B_D13: now also J3.7 (Pin_7)
- net B_D14: now also J3.5 (Pin_5)
- net B_D15: now also J3.3 (Pin_3)
- net B_D2: now also J3.8 (Pin_8)
- net B_D3: now also J3.10 (Pin_10)
- net B_D4: now also J3.12 (Pin_12)
- net B_D5: now also J3.14 (Pin_14)
- net B_D6: now also J3.16 (Pin_16)
- net B_D7: now also J3.18 (Pin_18)
- net B_D8: now also J3.17 (Pin_17)
- net B_D9: now also J3.15 (Pin_15)
- net B_~{RESET}: now also J3.1 (Pin_1)
- net GND: now also J3.19 (Pin_19), J3.2 (Pin_2), J3.22 (Pin_22), J3.24 (Pin_24), J3.26 (Pin_26), J3.28 (Pin_28), J3.30 (Pin_30), J3.40 (Pin_40), J3.43 (Pin_43)
- net IORDY: now also J3.27 (Pin_27)
- net I_A0: now also J3.35 (Pin_35)
- net I_A1: now also J3.33 (Pin_33)
- net I_A2: now also J3.36 (Pin_36)
- net VCC: now also F1.1
- net ~{DMACK}: now also J3.29 (Pin_29)
- net ~{IDE_ACT}: now also J3.39 (Pin_39)
- net ~{IDE_CS1}: now also J3.37 (Pin_37)
- net ~{IDE_CS2}: now also J3.38 (Pin_38)
- net ~{IDE_IRQ}: now also J3.31 (Pin_31)
- net ~{IORD}: now also J3.25 (Pin_25)
- net ~{IOWR}: now also J3.23 (Pin_23)
- new net: F1.2, J3.41 (Pin_41), J3.42 (Pin_42)
- new net A9: U5.16 (B2)

Commit message: PCB: Start routing PCB
Connections:
- net B_D0: now also U4.9 (A7); no longer U4.2 (A0)
- net B_D1: now also U4.7 (A5); no longer U4.3 (A1)
- net B_D10: now also U3.7 (A5); no longer U3.4 (A2)
- net B_D11: now also U3.9 (A7); no longer U3.5 (A3)
- net B_D12: now also U4.2 (A0); no longer U3.6 (A4)
- net B_D13: now also U4.4 (A2); no longer U3.7 (A5)
- net B_D14: now also U4.6 (A4); no longer U3.8 (A6)
- net B_D15: now also U4.8 (A6); no longer U3.9 (A7)
- net B_D2: now also U4.5 (A3); no longer U4.4 (A2)
- net B_D3: now also U4.3 (A1); no longer U4.5 (A3)
- net B_D4: now also U3.8 (A6); no longer U4.6 (A4)
- net B_D5: now also U3.6 (A4); no longer U4.7 (A5)
- net B_D6: now also U3.4 (A2); no longer U4.8 (A6)
- net B_D7: now also U3.2 (A0); no longer U4.9 (A7)
- net B_D8: now also U3.3 (A1); no longer U3.2 (A0)
- net B_D9: now also U3.5 (A3); no longer U3.3 (A1)
- net D0: now also U4.11 (B7); no longer U4.18 (B0)
- net D1: now also U4.13 (B5); no longer U4.17 (B1)
- net D10: now also U3.13 (B5); no longer U3.16 (B2)
- net D11: now also U3.11 (B7); no longer U3.15 (B3)
- net D12: now also U4.18 (B0); no longer U3.14 (B4)
- net D13: now also U4.16 (B2); no longer U3.13 (B5)
- net D14: now also U4.14 (B4); no longer U3.12 (B6)
- net D15: now also U4.12 (B6); no longer U3.11 (B7)
- net D2: now also U4.15 (B3); no longer U4.16 (B2)
- net D3: now also U4.17 (B1); no longer U4.15 (B3)
- net D4: now also U3.12 (B6); no longer U4.14 (B4)
- net D5: now also U3.14 (B4); no longer U4.13 (B5)
- net D6: now also U3.16 (B2); no longer U4.12 (B6)
- net D7: now also U3.18 (B0); no longer U4.11 (B7)
- net D8: now also U3.17 (B1); no longer U3.18 (B0)
- net D9: now also U3.15 (B3); no longer U3.17 (B1)
Changed lines of the file:
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@@
     (effects (font (size 1.27 1.27)) (justify right bottom))
   )
-  (label "B_D7" (at 105.41 102.235 0)
+  (label "B_D7" (at 105.41 29.845 0)
     (effects (font (size 1.27 1.27)) (justify left bottom))
   )
@@
     (effects (font (size 1.27 1.27)) (justify left bottom))
   )
-  (label "B_D0" (at 105.41 84.455 0)
-    (effects (font (size 1.27 1.27)) (justify left bottom))
-  )
-  (label "B_D9" (at 105.41 32.385 0)
+  (label "B_D0" (at 105.41 102.235 0)
+    (effects (font (size 1.27 1.27)) (justify left bottom))
+  )
+  (label "B_D9" (at 105.41 37.465 0)
     (effects (font (size 1.27 1.27)) (justify left bottom))
   )
@@
     (effects (font (size 1.27 1.27)) (justify left bottom))
   )
-  (label "D4" (at 80.01 94.615 180)
+  (label "D4" (at 80.01 45.085 180)
     (effects (font (size 1.27 1.27)) (justify right bottom))
   )
@@
     (effects (font (size 1.27 1.27)) (justify left bottom))
   )
-  (label "D11" (at 80.01 37.465 180)
+  (label "D11" (at 80.01 47.625 180)
     (effects (font (size 1.27 1.27)) (justify right bottom))
   )
@@
     (effects (font (size 1.27 1.27)) (justify right bottom))
   )
-  (label "B_D8" (at 105.41 29.845 0)
-    (effects (font (size 1.27 1.27)) (justify left bottom))
-  )
-  (label "B_D5" (at 105.41 97.155 0)
-    (effects (font (size 1.27 1.27)) (justify left bottom))
-  )
-  (label "B_D4" (at 105.41 94.615 0)
+  (label "B_D8" (at 105.41 32.385 0)
+    (effects (font (size 1.27 1.27)) (justify left bottom))
+  )
+  (label "B_D5" (at 105.41 40.005 0)
+    (effects (font (size 1.27 1.27)) (justify left bottom))
+  )
+  (label "B_D4" (at 105.41 45.085 0)
     (effects (font (size 1.27 1.27)) (justify left bottom))
   )
@@
     (effects (font (size 1.27 1.27)) (justify left bottom))
   )
-  (label "B_D10" (at 105.41 34.925 0)
-    (effects (font (size 1.27 1.27)) (justify left bottom))
-  )
-  (label "D13" (at 80.01 42.545 180)
+  (label "B_D10" (at 105.41 42.545 0)
+    (effects (font (size 1.27 1.27)) (justify left bottom))
+  )
+  (label "D13" (at 80.01 89.535 180)
     (effects (font (size 1.27 1.27)) (justify right bottom))
   )
@@
     (effects (font (size 1.27 1.27)) (justify right bottom))
   )
-  (label "B_D15" (at 105.41 47.625 0)
-    (effects (font (size 1.27 1.27)) (justify left bottom))
-  )
-  (label "D7" (at 80.01 102.235 180)
-    (effects (font (size 1.27 1.27)) (justify right bottom))
-  )
-  (label "D14" (at 80.01 45.085 180)
-    (effects (font (size 1.27 1.27)) (justify right bottom))
-  )
-  (label "B_D14" (at 105.41 45.085 0)
-    (effects (font (size 1.27 1.27)) (justify left bottom))
-  )
-  (label "D3" (at 80.01 92.075 180)
-    (effects (font (size 1.27 1.27)) (justify right bottom))
-  )
-  (label "D15" (at 80.01 47.625 180)
+  (label "B_D15" (at 105.41 99.695 0)
+    (effects (font (size 1.27 1.27)) (justify left bottom))
+  )
+  (label "D7" (at 80.01 29.845 180)
+    (effects (font (size 1.27 1.27)) (justify right bottom))
+  )
+  (label "D14" (at 80.01 94.615 180)
+    (effects (font (size 1.27 1.27)) (justify right bottom))
+  )
+  (label "B_D14" (at 105.41 94.615 0)
+    (effects (font (size 1.27 1.27)) (justify left bottom))
+  )
+  (label "D3" (at 80.01 86.995 180)
+    (effects (font (size 1.27 1.27)) (justify right bottom))
+  )
+  (label "D15" (at 80.01 99.695 180)
     (effects (font (size 1.27 1.27)) (justify right bottom))
   )
@@
     (effects (font (size 1.27 1.27)) (justify right bottom))
   )
-  (label "B_D1" (at 105.41 86.995 0)
+  (label "B_D1" (at 105.41 97.155 0)
     (effects (font (size 1.27 1.27)) (justify left bottom))
   )
@@
     (effects (font (size 1.27 1.27)) (justify right bottom))
   )
-  (label "D8" (at 80.01 29.845 180)
-    (effects (font (size 1.27 1.27)) (justify right bottom))
-  )
-  (label "D5" (at 80.01 97.155 180)
+  (label "D8" (at 80.01 32.385 180)
+    (effects (font (size 1.27 1.27)) (justify right bottom))
+  )
+  (label "D5" (at 80.01 40.005 180)
     (effects (font (size 1.27 1.27)) (justify right bottom))
   )
@@
     (effects (font (size 1.27 1.27)) (justify right bottom))
   )
-  (label "D0" (at 80.01 84.455 180)
+  (label "D0" (at 80.01 102.235 180)
     (effects (font (size 1.27 1.27)) (justify right bottom))
   )
@@
     (effects (font (size 1.27 1.27)) (justify left bottom))
   )
-  (label "D2" (at 80.01 89.535 180)
-    (effects (font (size 1.27 1.27)) (justify right bottom))
-  )
-  (label "B_D13" (at 105.41 42.545 0)
+  (label "D2" (at 80.01 92.075 180)
+    (effects (font (size 1.27 1.27)) (justify right bottom))
+  )
+  (label "B_D13" (at 105.41 89.535 0)
     (effects (font (size 1.27 1.27)) (justify left bottom))
   )
@@
     (effects (font (size 1.27 1.27)) (justify right bottom))
   )
-  (label "D10" (at 80.01 34.925 180)
+  (label "D10" (at 80.01 42.545 180)
     (effects (font (size 1.27 1.27)) (justify right bottom))
   )
@@
     (effects (font (size 1.27 1.27)) (justify right bottom))
   )
-  (label "B_D6" (at 105.41 99.695 0)
+  (label "B_D6" (at 105.41 34.925 0)
     (effects (font (size 1.27 1.27)) (justify left bottom))
   )
@@
     (effects (font (size 1.27 1.27)) (justify right bottom))
   )
-  (label "B_D12" (at 105.41 40.005 0)
-    (effects (font (size 1.27 1.27)) (justify left bottom))
-  )
-  (label "D12" (at 80.01 40.005 180)
+  (label "B_D12" (at 105.41 84.455 0)
+    (effects (font (size 1.27 1.27)) (justify left bottom))
+  )
+  (label "D12" (at 80.01 84.455 180)
     (effects (font (size 1.27 1.27)) (justify right bottom))
   )
@@
     (effects (font (size 1.27 1.27)) (justify right bottom))
   )
-  (label "B_D3" (at 105.41 92.075 0)
-    (effects (font (size 1.27 1.27)) (justify left bottom))
-  )
-  (label "D6" (at 80.01 99.695 180)
-    (effects (font (size 1.27 1.27)) (justify right bottom))
-  )
-  (label "D9" (at 80.01 32.385 180)
+  (label "B_D3" (at 105.41 86.995 0)
+    (effects (font (size 1.27 1.27)) (justify left bottom))
+  )
+  (label "D6" (at 80.01 34.925 180)
+    (effects (font (size 1.27 1.27)) (justify right bottom))
+  )
+  (label "D9" (at 80.01 37.465 180)
     (effects (font (size 1.27 1.27)) (justify right bottom))
   )
@@
     (effects (font (size 1.27 1.27)) (justify right bottom))
   )
-  (label "B_D11" (at 105.41 37.465 0)
+  (label "B_D11" (at 105.41 47.625 0)
     (effects (font (size 1.27 1.27)) (justify left bottom))
   )
@@
     (effects (font (size 1.27 1.27)) (justify left bottom))
   )
-  (label "B_D2" (at 105.41 89.535 0)
-    (effects (font (size 1.27 1.27)) (justify left bottom))
-  )
-  (label "D1" (at 80.01 86.995 180)
-    (effects (font (size 1.27 1.27)) (justify right bottom))
-  )
+  (label "B_D2" (at 105.41 92.075 0)
+    (effects (font (size 1.27 1.27)) (justify left bottom))
+  )
+  (label "D1" (at 80.01 97.155 180)
+    (effects (font (size 1.27 1.27)) (justify right bottom))
+  )

Commit message: PCB: Keep on routing...
Changed lines of the file:
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@@
-    (stroke (width 0) (type default) (color 0 0 0 0))
-  )
-  (wire (pts (xy 184.785 103.505) (xy 153.67 103.505))
     (stroke (width 0) (type default) (color 0 0 0 0))
   )
@@
     (stroke (width 0) (type default) (color 0 0 0 0))
   )
-  (wire (pts (xy 153.67 103.505) (xy 153.67 56.515))
-    (stroke (width 0) (type default) (color 0 0 0 0))
-  )
   (bus (pts (xy 212.09 65.405) (xy 212.09 67.945))
     (stroke (width 0) (type default) (color 0 0 0 0))
@@
   )
   (wire (pts (xy 76.835 154.305) (xy 80.01 154.305))
-    (stroke (width 0) (type default) (color 0 0 0 0))
-  )
-  (wire (pts (xy 153.67 56.515) (xy 219.075 56.515))
     (stroke (width 0) (type default) (color 0 0 0 0))
   )
@@
     (effects (font (size 1.27 1.27)) (justify right))
   )
-  (hierarchical_label "~{IDE_IRQ}" (shape output) (at 219.075 56.515 0)
-    (effects (font (size 1.27 1.27)) (justify left))
-  )
   (symbol (lib_id "power:VCC") (at 92.71 139.065 0) (unit 1)

Commit message: PCB: More work...
* Add DIP Switches for Ram/Rom/IDE config
* Route bank select signals for Flash rom
* Flip IDE to bottom of the board
* Add some bulk capacitors
Parts:
- F1: LCSC # (none) -> C210831
- J2: footprint Connector_PinHeader_2.54mm:PinHeader_1x02_P2.54mm_Vertical -> Connector_PinHeader_2.00mm:PinHeader_1x02_P2.00mm_Vertical
Changed lines of the file:
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@@
+      (effects (font (size 1.27 1.27)) hide)
+    )
+    (property "LCSC #" "C210831" (id 4) (at 222.25 113.03 0)
       (effects (font (size 1.27 1.27)) hide)
     )
@@
       (effects (font (size 1.27 1.27)) (justify right))
     )
-    (property "Footprint" "Connector_PinHeader_2.54mm:PinHeader_1x02_P2.54mm_Vertical" (id 2) (at 128.27 146.685 0)
+    (property "Footprint" "Connector_PinHeader_2.00mm:PinHeader_1x02_P2.00mm_Vertical" (id 2) (at 128.27 146.685 0)
       (effects (font (size 1.27 1.27)) hide)
     )

Commit message: PCB: Route Flash bank switch jumper
Connections:
- no-connect marks 6 -> 7
Changed lines of the file:
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@@
   (no_connect (at 197.485 103.505))
   (no_connect (at 197.485 106.045))
+  (no_connect (at 197.485 118.745))
   (no_connect (at 197.485 88.265))
   (bus_entry (at 73.025 97.155) (size 2.54 2.54)
@@
     (effects (font (size 1.27 1.27)) (justify right bottom))
   )
-  (label "~{RESET}" (at 80.01 164.465 180)
+  (label "~{RST}" (at 80.01 164.465 180)
     (effects (font (size 1.27 1.27)) (justify right bottom))
   )

Commit message: PCB: Add 22 Ohm series resistors for SDRAM
Parts:
- F1: LCSC # C210831 -> C151162
Changed lines of the file:
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@@
       (effects (font (size 1.27 1.27)) hide)
     )
-    (property "LCSC #" "C210831" (id 4) (at 222.25 113.03 0)
+    (property "LCSC #" "C151162" (id 4) (at 222.25 113.03 0)
       (effects (font (size 1.27 1.27)) hide)
     )

Commit message: PCB: Remove useless cfgin connection
Parts:
- removed R8: 10K, Resistor_SMD:R_0603_1608Metric, symbol Device:R
- added R6, R7: 10K, Resistor_SMD:R_0603_1608Metric, symbol Device:R
- renumbered J2 to J3, J3 to J4, R5 to R3, R6 to R4, R7 to R5, R9 to R8, R10 to R9
Connections:
- net GND: now also J4.44 (Pin_44)
- net VCC: now also R6.2, R7.2
- net ~{DMACK}: now also R6.1
- net ~{IDE_IRQ}: now also R7.1
- no-connect marks 7 -> 6
