File: Kicad/RAM.kicad_sch (KiCad schematic)
At the start: 17 parts, among them U6 74LVC245, U7 74LVC245, U8 MT48LC8M16A2P

Commit message: PCB: Remove useless cfgin connection
Parts:
- renumbered C17 to C16, C18 to C17, C19 to C18, C20 to C19, C21 to C20, C22 to C21, C23 to C22, C24 to C23, C25 to C24, U7 to U6, U6 to U7
Changed lines of the file:
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@@
   (symbol (lib_id "Device:C_Small") (at 156.21 186.69 0) (unit 1)
     (in_bom yes) (on_board yes) (fields_autoplaced)
-    (property "Reference" "C24" (id 0) (at 158.75 185.4199 0)
+    (property "Reference" "C23" (id 0) (at 158.75 185.4199 0)
       (effects (font (size 1.27 1.27)) (justify left))
     )
@@
   (symbol (lib_id "Device:C_Small") (at 93.98 186.69 0) (unit 1)
     (in_bom yes) (on_board yes) (fields_autoplaced)
-    (property "Reference" "C17" (id 0) (at 96.52 185.4199 0)
+    (property "Reference" "C16" (id 0) (at 96.52 185.4199 0)
       (effects (font (size 1.27 1.27)) (justify left))
     )
@@
   (symbol (lib_id "74xx:74HC245") (at 99.06 102.87 0) (mirror y) (unit 1)
     (in_bom yes) (on_board yes)
-    (property "Reference" "U6" (id 0) (at 105.41 86.36 0))
+    (property "Reference" "U7" (id 0) (at 105.41 86.36 0))
     (property "Value" "74LVC245" (id 1) (at 104.14 119.38 0))
     (property "Footprint" "Package_SO:TSSOP-20_4.4x6.5mm_P0.65mm" (id 2) (at 99.06 102.87 0)
@@
   (symbol (lib_id "Device:C_Small") (at 129.54 186.69 0) (unit 1)
     (in_bom yes) (on_board yes) (fields_autoplaced)
-    (property "Reference" "C21" (id 0) (at 132.08 185.4199 0)
+    (property "Reference" "C20" (id 0) (at 132.08 185.4199 0)
       (effects (font (size 1.27 1.27)) (justify left))
     )
@@
   (symbol (lib_id "power:+3.3V") (at 99.06 29.21 0) (unit 1)
     (in_bom yes) (on_board yes) (fields_autoplaced)
-    (property "Reference" "#PWR042" (id 0) (at 99.06 33.02 0)
+    (property "Reference" "#PWR041" (id 0) (at 99.06 33.02 0)
       (effects (font (size 1.27 1.27)) hide)
     )
@@
   (symbol (lib_id "Device:C_Small") (at 147.32 186.69 0) (unit 1)
     (in_bom yes) (on_board yes) (fields_autoplaced)
-    (property "Reference" "C23" (id 0) (at 149.86 185.4199 0)
+    (property "Reference" "C22" (id 0) (at 149.86 185.4199 0)
       (effects (font (size 1.27 1.27)) (justify left))
     )
@@
   (symbol (lib_id "Device:C_Small") (at 120.65 186.69 0) (unit 1)
     (in_bom yes) (on_board yes) (fields_autoplaced)
-    (property "Reference" "C20" (id 0) (at 123.19 185.4199 0)
+    (property "Reference" "C19" (id 0) (at 123.19 185.4199 0)
       (effects (font (size 1.27 1.27)) (justify left))
     )
@@
   (symbol (lib_id "power:+3.3V") (at 99.06 82.55 0) (unit 1)
     (in_bom yes) (on_board yes) (fields_autoplaced)
-    (property "Reference" "#PWR044" (id 0) (at 99.06 86.36 0)
+    (property "Reference" "#PWR043" (id 0) (at 99.06 86.36 0)
       (effects (font (size 1.27 1.27)) hide)
     )
@@
   (symbol (lib_id "74xx:74HC245") (at 99.06 49.53 0) (mirror y) (unit 1)
     (in_bom yes) (on_board yes)
-    (property "Reference" "U7" (id 0) (at 105.41 33.02 0))
+    (property "Reference" "U6" (id 0) (at 105.41 33.02 0))
     (property "Value" "74LVC245" (id 1) (at 104.14 66.04 0))
     (property "Footprint" "Package_SO:TSSOP-20_4.4x6.5mm_P0.65mm" (id 2) (at 99.06 49.53 0)
@@
   (symbol (lib_id "power:GND") (at 99.06 123.19 0) (unit 1)
     (in_bom yes) (on_board yes) (fields_autoplaced)
-    (property "Reference" "#PWR045" (id 0) (at 99.06 129.54 0)
+    (property "Reference" "#PWR044" (id 0) (at 99.06 129.54 0)
       (effects (font (size 1.27 1.27)) hide)
     )
@@
   (symbol (lib_id "Device:C_Small") (at 102.87 186.69 0) (unit 1)
     (in_bom yes) (on_board yes) (fields_autoplaced)
-    (property "Reference" "C18" (id 0) (at 105.41 185.4199 0)
+    (property "Reference" "C17" (id 0) (at 105.41 185.4199 0)
       (effects (font (size 1.27 1.27)) (justify left))
     )
@@
   (symbol (lib_id "power:GND") (at 99.06 69.85 0) (unit 1)
     (in_bom yes) (on_board yes) (fields_autoplaced)
-    (property "Reference" "#PWR043" (id 0) (at 99.06 76.2 0)
+    (property "Reference" "#PWR042" (id 0) (at 99.06 76.2 0)
       (effects (font (size 1.27 1.27)) hide)
     )
@@
   (symbol (lib_id "power:+3.3V") (at 170.815 101.6 0) (unit 1)
     (in_bom yes) (on_board yes) (fields_autoplaced)
-    (property "Reference" "#PWR048" (id 0) (at 170.815 105.41 0)
+    (property "Reference" "#PWR047" (id 0) (at 170.815 105.41 0)
       (effects (font (size 1.27 1.27)) hide)
     )
@@
   (symbol (lib_id "Device:C_Small") (at 111.76 186.69 0) (unit 1)
     (in_bom yes) (on_board yes) (fields_autoplaced)
-    (property "Reference" "C19" (id 0) (at 114.3 185.4199 0)
+    (property "Reference" "C18" (id 0) (at 114.3 185.4199 0)
       (effects (font (size 1.27 1.27)) (justify left))
     )
@@
   (symbol (lib_id "Device:C_Small") (at 138.43 186.69 0) (unit 1)
     (in_bom yes) (on_board yes) (fields_autoplaced)
-    (property "Reference" "C22" (id 0) (at 140.97 185.4199 0)
+    (property "Reference" "C21" (id 0) (at 140.97 185.4199 0)
       (effects (font (size 1.27 1.27)) (justify left))
     )
@@
   (symbol (lib_id "power:GND") (at 156.845 61.595 0) (unit 1)
     (in_bom yes) (on_board yes) (fields_autoplaced)
-    (property "Reference" "#PWR046" (id 0) (at 156.845 67.945 0)
+    (property "Reference" "#PWR045" (id 0) (at 156.845 67.945 0)
       (effects (font (size 1.27 1.27)) hide)
     )
@@
   (symbol (lib_id "Device:C_Small") (at 166.37 186.69 0) (unit 1)
     (in_bom yes) (on_board yes) (fields_autoplaced)
-    (property "Reference" "C25" (id 0) (at 168.91 185.4199 0)
+    (property "Reference" "C24" (id 0) (at 168.91 185.4199 0)
       (effects (font (size 1.27 1.27)) (justify left))
     )
@@
   (symbol (lib_id "power:GND") (at 166.37 189.23 0) (unit 1)
     (in_bom yes) (on_board yes)
-    (property "Reference" "#PWR047" (id 0) (at 166.37 195.58 0)
+    (property "Reference" "#PWR046" (id 0) (at 166.37 195.58 0)
       (effects (font (size 1.27 1.27)) hide)
     )
@@
   (symbol (lib_id "power:+3.3V") (at 86.995 184.15 0) (unit 1)
     (in_bom yes) (on_board yes) (fields_autoplaced)
-    (property "Reference" "#PWR041" (id 0) (at 86.995 187.96 0)
+    (property "Reference" "#PWR040" (id 0) (at 86.995 187.96 0)
       (effects (font (size 1.27 1.27)) hide)
     )
@@
   (symbol (lib_id "power:GND") (at 193.675 121.285 0) (unit 1)
     (in_bom yes) (on_board yes)
-    (property "Reference" "#PWR049" (id 0) (at 193.675 127.635 0)
-      (effects (font (size 1.27 1.27)) hide)
-    )
+    (property "Reference" "#PWR048" (id 0) (at 193.675 127.635 0)
+      (effects (font (size 1.27 1.27)) hide)
+    )

Commit message: PCB: Fixups
* Tweak KEL connector hole sizes
* Fixup MT48LC8M16A2P - Had copied this from the 16M16 part and forgot to make A12 an NC
Parts:
- RN2, RN3, RN4, RN5: value R_Pack04 -> 22
Other:
- company: (none) -> Matt Harlum
- title: (none) -> CIDER
Changed lines of the file:
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@@
 (kicad_sch (version 20211123) (generator eeschema)
   (paper "A4")
+  (title_block
+    (title "CIDER")
+    (company "Matt Harlum")
+  )
   (junction (at 120.65 189.23) (diameter 1.016) (color 0 0 0 0)
   )
@@
     (in_bom yes) (on_board yes)
     (property "Reference" "RN4" (id 0) (at 118.745 87.63 90))
-    (property "Value" "R_Pack04" (id 1) (at 118.745 86.36 90)
-      (effects (font (size 1.27 1.27)) hide)
-    )
+    (property "Value" "22" (id 1) (at 118.745 85.725 90))
     (property "Footprint" "Resistor_SMD:R_Array_Convex_4x0603" (id 2) (at 118.745 85.725 90)
       (effects (font (size 1.27 1.27)) hide)
@@
     (in_bom yes) (on_board yes)
     (property "Reference" "RN3" (id 0) (at 118.745 57.15 90))
-    (property "Value" "R_Pack04" (id 1) (at 118.745 43.18 90)
-      (effects (font (size 1.27 1.27)) hide)
-    )
+    (property "Value" "22" (id 1) (at 114.935 57.15 90))
     (property "Footprint" "Resistor_SMD:R_Array_Convex_4x0603" (id 2) (at 118.745 42.545 90)
       (effects (font (size 1.27 1.27)) hide)
@@
     (in_bom yes) (on_board yes)
     (property "Reference" "RN5" (id 0) (at 118.745 110.49 90))
-    (property "Value" "R_Pack04" (id 1) (at 118.745 96.52 90)
-      (effects (font (size 1.27 1.27)) hide)
-    )
+    (property "Value" "22" (id 1) (at 122.555 111.125 90))
     (property "Footprint" "Resistor_SMD:R_Array_Convex_4x0603" (id 2) (at 118.745 95.885 90)
       (effects (font (size 1.27 1.27)) hide)
@@
     (in_bom yes) (on_board yes)
     (property "Reference" "RN2" (id 0) (at 118.745 34.29 90))
-    (property "Value" "R_Pack04" (id 1) (at 118.745 33.02 90)
-      (effects (font (size 1.27 1.27)) hide)
-    )
+    (property "Value" "22" (id 1) (at 118.745 32.385 90))
     (property "Footprint" "Resistor_SMD:R_Array_Convex_4x0603" (id 2) (at 118.745 32.385 90)
       (effects (font (size 1.27 1.27)) hide)
@@
     (pin "1")
   )
-  (symbol (lib_id "MT48LC8M16A2P:MT48LC8M16A2P") (at 182.88 64.77 0) (unit 1)
+  (symbol (lib_name "MT48LC8M16A2P_1") (lib_id "MT48LC8M16A2P:MT48LC8M16A2P") (at 182.88 64.77 0) (unit 1)
     (in_bom yes) (on_board yes) (fields_autoplaced)
     (property "Reference" "U8" (id 0) (at 182.88 29.21 0))

Commit message: Fixup some of the JLC part numbers
Parts:
- U8: LCSC # C367430 -> C62379
Changed lines of the file:
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@@
       (effects (font (size 1.27 1.27)) hide)
     )
-    (property "LCSC #" "C367430" (id 4) (at 182.245 64.77 0)
+    (property "LCSC #" "C62379" (id 4) (at 182.245 64.77 0)
       (effects (font (size 1.27 1.27)) hide)
     )
@@
       (effects (font (size 1.27 1.27)) hide)
     )
-    (property "LCSC #" "C367430" (id 4) (at 182.88 64.77 0)
+    (property "LCSC #" "C62379" (id 4) (at 182.88 64.77 0)
       (effects (font (size 1.27 1.27)) hide)
     )
