File: Kicad/Amiga-CPLD.kicad_sch (KiCad schematic)
At the start: 27 parts, among them CN1 CDTV-DIAG, J1 JTAG, J2 LED, J3 A500_MODE, J5 To JP15, SW1 SW_DIP_x04, U1 AZ1117-3.3, U11 74LVC1G32, U2 XC95144XL-TQ100, X1 50MHz

Commit message: Rev_A1: Add pull-down resistor for U11 input, add tooling holes
Parts:
- added R12: 10K, Resistor_SMD:R_0603_1608Metric, symbol Device:R
Connections:
- net GND: now also R12.1
- net at J5.2 (Pin_2), U11.2: now also R12.2
- net NOEXT renamed A500
Changed lines of the file:
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@@
   (junction (at 34.29 128.27) (diameter 0) (color 0 0 0 0)
+  )
+  (junction (at 238.76 121.92) (diameter 0) (color 0 0 0 0)
   )
   (junction (at 225.425 68.58) (diameter 0) (color 0 0 0 0)
@@
     (effects (font (size 1.27 1.27)) (justify right bottom))
   )
-  (label "NOEXT" (at 255.27 91.44 180)
+  (label "A500" (at 255.27 91.44 180)
     (effects (font (size 1.27 1.27)) (justify right bottom))
   )
@@
     (effects (font (size 1.27 1.27)) (justify left bottom))
   )
-  (label "NOEXT" (at 133.35 31.75 180)
+  (label "A500" (at 133.35 31.75 180)
     (effects (font (size 1.27 1.27)) (justify right bottom))
   )
@@
     )
     (pin "1")
+  )
+  (symbol (lib_id "Device:R") (at 238.76 125.73 180) (unit 1)
+    (in_bom yes) (on_board yes)
+    (property "Reference" "R12" (id 0) (at 233.68 125.73 90))
+    (property "Value" "10K" (id 1) (at 236.22 125.73 90))
+    (property "Footprint" "Resistor_SMD:R_0603_1608Metric" (id 2) (at 240.538 125.73 90)
+      (effects (font (size 1.27 1.27)) hide)
+    )
+    (property "Datasheet" "~" (id 3) (at 238.76 125.73 0)
+      (effects (font (size 1.27 1.27)) hide)
+    )
+    (property "LCSC #" "C25804" (id 4) (at 238.76 125.73 90)
+      (effects (font (size 1.27 1.27)) hide)
+    )
+    (pin "1")
+    (pin "2")
   )
   (symbol (lib_id "power:+3.3V") (at 166.37 19.05 0) (unit 1)
@@
     (pin "2")
   )
+  (symbol (lib_id "power:GND") (at 238.76 129.54 0) (unit 1)
+    (in_bom yes) (on_board yes) (fields_autoplaced)
+    (property "Reference" "#PWR065" (id 0) (at 238.76 135.89 0)
+      (effects (font (size 1.27 1.27)) hide)
+    )
+    (property "Value" "GND" (id 1) (at 238.76 134.62 0))
+    (property "Footprint" "" (id 2) (at 238.76 129.54 0)
+      (effects (font (size 1.27 1.27)) hide)
+    )
+    (property "Datasheet" "" (id 3) (at 238.76 129.54 0)
+      (effects (font (size 1.27 1.27)) hide)
+    )
+    (pin "1")
+  )
 )

Commit message: Rev_A1: Fixup JLC Part # for Volt reg
Parts:
- U1: value AZ1117-3.3 -> AZ1117CR-3.3; LCSC # C362111 -> C460428
Changed lines of the file:
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@@
     (in_bom yes) (on_board yes) (fields_autoplaced)
     (property "Reference" "U1" (id 0) (at 93.98 151.5618 0))
-    (property "Value" "AZ1117-3.3" (id 1) (at 93.98 154.1018 0))
+    (property "Value" "AZ1117CR-3.3" (id 1) (at 93.98 154.1018 0))
     (property "Footprint" "Package_TO_SOT_SMD:SOT-89-3" (id 2) (at 93.98 151.765 0)
       (effects (font (size 1.27 1.27) italic) hide)
@@
       (effects (font (size 1.27 1.27)) hide)
     )
-    (property "LCSC #" " C362111" (id 4) (at 93.98 158.115 0)
+    (property "LCSC #" "C460428" (id 4) (at 93.98 158.115 0)
       (effects (font (size 1.27 1.27)) hide)
     )
